File: Clock.kicad_sch (KiCad schematic)
At the start: 24 parts, among them SW1 SW_Push, SW2 SW_SPDT, U1 LM555xM, U2 LM555xM, U3 LM555xM, U4 74LS08, U5 74LS04, U6 74LS32

Commit message: Added the ALU and flags register schematic.
Other:
- title: (none) -> 8 bit PC
Changed lines of the file:
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@@
 	(generator_version "9.0")
 	(paper "A4")
+	(title_block
+		(title "8 bit PC")
+		(date "2025-10-14")
+		(rev "1")
+	)
 	(junction
 		(at 264.16 33.02)
