File: PCB/_autosave-8-Bit-PC.kicad_pcb (KiCad board)
At the start: 2 copper layers, 279 parts, among them J1 USB_C_Receptacle_PowerOnly_6P, SW1 SW_Push, SW2 SW_SPDT, SW3 SW_DIP_x04, SW4 SW_SPDT, SW5 SW_DIP_x08, SW6 SW_Push, SW7 SW_SPDT, SW8 SW_Push, U1 LM555xM, U10 74LS08, U11 74LS02, U117 74LS245, U118 74ls245, U119 74LS173, U12 74LS173, U13 74LS283, U14 74LS283, U15 74LS86, U16 74LS86, U17 74LS245, U18 74LS157, U19 74LS173, U2 LM555xM, U20 74LS04, U21 74189, U22 74LS04, U23 74189, U24 74LS158, U25 74LS245, U26 74LS00, U27 74LS04, U28 74LS04, U29 74LS245, U3 LM555xM, U30 74LS161, U31 LM555xM, U32 74LS76, U33 74LS139, U34 D148K, U35 D148K, U36 D148K, U37 D148K, U38 74LS273, U39 74LS08, U4 74LS08, U40 AT28C64B-15PU, U41 74LS161, U42 74LS138, U43 AT28C64B-15PU, U44 AT28C64B-15PU, U45 74LS00, U46 74LS04, U47 74LS04, U48 74LS245, U49 74LS173, U5 74LS04, U50 74LS173, U51 74LS158, U52 74LS158, U6 74LS32, U7 74LS245, U8 74LS173, U9 74LS173

Commit message: added more models to work with on my pcb
Parts:
- R37, R38, R39, R61, R62, R63: moved to B.Cu
- moved C14 122.9 mm to (429.0, 343.5), turned to -90 degrees
- moved D31 87.4 mm to (337.6, 361.8), turned to 90 degrees
- moved D26 85.6 mm to (337.6, 386.8), turned to 90 degrees
- moved D32 83.0 mm to (337.6, 356.8), turned to 90 degrees
- moved D33 79.1 mm to (337.6, 351.8), turned to 90 degrees
- moved D27 79.1 mm to (337.6, 381.8), turned to 90 degrees
- moved D28 72.9 mm to (337.6, 376.8), turned to 90 degrees
- moved D60 67.0 mm to (77.0, 102.0)
- moved D61 67.0 mm to (83.0, 102.0)
- moved D59 67.0 mm to (71.0, 102.0)
- moved D29 67.0 mm to (337.6, 371.8), turned to 90 degrees
- moved U34 66.5 mm to (23.4, 382.0), turned to 90 degrees
- moved R24 66.1 mm to (342.5, 386.8)
- moved R31 65.3 mm to (342.5, 351.8)
- moved SW6 64.9 mm to (317.0, 378.5), turned to 180 degrees
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