File: PCB/8-Bit-PC.kicad_pcb (KiCad board)
At the start: 2 copper layers, 279 parts, among them J1 USB_C_Receptacle_PowerOnly_6P, SW1 SW_Push, SW2 SW_SPDT, SW3 SW_DIP_x04, SW4 SW_SPDT, SW5 SW_DIP_x08, SW6 SW_Push, SW7 SW_SPDT, SW8 SW_Push, U1 LM555xM, U10 74LS08, U11 74LS02, U117 74LS245, U118 74ls245, U119 74LS173, U12 74LS173, U13 74LS283, U14 74LS283, U15 74LS86, U16 74LS86, U17 74LS245, U18 74LS157, U19 74LS173, U2 LM555xM, U20 74LS04, U21 74189, U22 74LS04, U23 74189, U24 74LS158, U25 74LS245, U26 74LS00, U27 74LS04, U28 74LS04, U29 74LS245, U3 LM555xM, U30 74LS161, U31 LM555xM, U32 74LS76, U33 74LS139, U34 D148K, U35 D148K, U36 D148K, U37 D148K, U38 74LS273, U39 74LS08, U4 74LS08, U40 AT28C64B-15PU, U41 74LS161, U42 74LS138, U43 AT28C64B-15PU, U44 AT28C64B-15PU, U45 74LS00, U46 74LS04, U47 74LS04, U48 74LS245, U49 74LS173, U5 74LS04, U50 74LS173, U51 74LS158, U52 74LS158, U6 74LS32, U7 74LS245, U8 74LS173, U9 74LS173

Commit message: got the PCB layed out into one group and started routing the traces and fixing DRC errors.
Parts:
- R77, R78, R79, R80: moved to B.Cu
- moved R1 319.2 mm to (293.0, 127.4)
- moved C2 319.2 mm to (275.6, 154.4)
- moved C3 319.2 mm to (275.6, 149.7)
- moved C4 319.2 mm to (293.3, 134.2)
- moved C5 319.2 mm to (301.1, 136.0)
- moved C6 319.2 mm to (301.1, 131.9)
- moved D1 319.2 mm to (271.3, 134.9)
- moved R3 319.2 mm to (275.5, 139.2)
- moved R4 319.2 mm to (282.1, 157.5)
- moved R5 319.2 mm to (292.6, 157.5)
- moved R6 319.2 mm to (296.3, 147.2)
- moved SW1 319.2 mm to (283.1, 131.2)
- moved SW2 319.2 mm to (301.3, 151.9)
- moved U2 319.2 mm to (282.6, 144.7)
- moved U3 319.2 mm to (290.1, 144.7)
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Routing:
- net BUS_5: track 0.00 -> 48.2 mm
Other:
- board outline added: 320.5 x 165.5 mm

Commit message: Routed the traces for the ground
Parts:
- SW2, SW4, SW7: footprint Button_Switch_SMD:SW_SPDT_CK_JS102011SAQN -> Button_Switch_THT:SW_Slide_SPDT_Straight_CK_OS102011MS2Q
- U16, U6: footprint footprints:N14 -> Package_DIP:DIP-14_W7.62mm
- U21, U23: value 74189 -> 74F189SC; footprint Custom:N16 -> Custom:SOIC16_9P9X3P9_ONS
- moved U16 28.1 mm to (289.4, 112.8), turned to 90 degrees
- moved U23 5.68 mm to (198.7, 117.6)
- moved C7 4.83 mm to (317.6, 107.0)
- moved R2 4.83 mm to (309.5, 111.5)
- moved RV1 4.83 mm to (320.8, 109.0)
- moved U21 4.59 mm to (190.2, 117.6)
- moved SW4 1.90 mm to (261.0, 23.5)
- moved SW2 1.84 mm to (302.8, 153.0)
Connections:
- C12 pad 2: BUS_5 -> GND
- C13 pad 2: BUS_5 -> GND
- D19 pad 2: Net-(D18-A) -> Net-(D19-A)
- D24 pad 1: BUS_5 -> /MAR/PROG
- D66 pad 2: BUS_5 -> BUS_4
- D68 pad 2: BUS_5 -> BUS_6
- D69 pad 2: BUS_5 -> BUS_7
- R24 pad 2: BUS_5 -> GND
- R25 pad 2: BUS_5 -> GND
- R26 pad 2: BUS_5 -> GND
- R27 pad 2: BUS_5 -> GND
- R28 pad 2: BUS_5 -> GND
- R29 pad 2: BUS_5 -> GND
- R30 pad 2: BUS_5 -> GND
- R31 pad 2: BUS_5 -> GND
- R32 pad 2: BUS_5 -> GND
- R73 pad 1: BUS_5 -> BUS_7
- R74 pad 1: BUS_5 -> BUS_6
- R76 pad 1: BUS_5 -> BUS_4
- SW3 pad 1: BUS_5 -> /MAR/PROG
- SW3 pad 2: BUS_5 -> /MAR/PROG
- SW3 pad 5: BUS_5 -> /MAR/PROG
- SW3 pad 6: BUS_5 -> /MAR/PROG
- SW4 pad 1: BUS_5 -> /MAR/PROG
- SW5 pad 10: BUS_5 -> Net-(U52-I0b)
- SW5 pad 11: BUS_5 -> GND
- SW5 pad 12: BUS_5 -> GND
- SW5 pad 15: BUS_5 -> GND
- SW5 pad 16: BUS_5 -> GND
- SW5 pad 3: BUS_5 -> GND
- SW5 pad 4: BUS_5 -> GND
- SW5 pad 5: BUS_5 -> Net-(U52-I0d)
- SW5 pad 6: BUS_5 -> Net-(U52-I0c)
- SW5 pad 7: BUS_5 -> GND
- SW5 pad 8: BUS_5 -> GND
- SW5 pad 9: BUS_5 -> Net-(U52-I0a)
- SW6 pad 1: BUS_5 -> GND
- U11 pad 11: Net-(U14-S2) -> Net-(D18-A)
- U11 pad 12: Net-(D18-A) -> Net-(D19-A)
- U117 pad 10: unconnected-(U117-GND-Pad10) -> GND
- U117 pad 15: BUS_5 -> BUS_4
- U117 pad 17: BUS_5 -> BUS_6
- U117 pad 18: BUS_5 -> BUS_7
- U117 pad 2: IR_7 -> IR_4
- U117 pad 20: unconnected-(U117-VCC-Pad20) -> VCC
- U117 pad 3: IR_6 -> IR_5
- U117 pad 4: IR_5 -> IR_6
- U117 pad 5: IR_4 -> IR_7
- U117 pad 6: Net-(D116-A) -> Net-(D119-A)
- U117 pad 7: Net-(D117-A) -> Net-(D118-A)
- U117 pad 8: Net-(D118-A) -> Net-(D117-A)
- U117 pad 9: Net-(D119-A) -> Net-(D116-A)
- U118 pad 11: BUS_5 -> BUS_4
- U118 pad 13: BUS_5 -> BUS_6
- U118 pad 14: BUS_5 -> BUS_7
- U118 pad 16: unconnected-(U118-VCC-Pad16) -> VCC
- U118 pad 3: IR_4 -> IR_7
- U118 pad 4: IR_5 -> IR_6
- U118 pad 5: IR_6 -> IR_5
- U118 pad 6: IR_7 -> IR_4
- U118 pad 8: unconnected-(U118-GND-Pad8) -> GND
- U119 pad 16: unconnected-(U119-VCC-Pad16) -> VCC
- U119 pad 3: Net-(D119-A) -> Net-(D116-A)
- U119 pad 4: Net-(D118-A) -> Net-(D117-A)
- U119 pad 5: Net-(D117-A) -> Net-(D118-A)
- U119 pad 6: Net-(D116-A) -> Net-(D119-A)
- U119 pad 8: unconnected-(U119-GND-Pad8) -> GND
- U12 pad 16: unconnected-(U12-VCC-Pad16) -> VCC
- U12 pad 8: unconnected-(U12-GND-Pad8) -> GND
- U13 pad 16: unconnected-(U13-VCC-Pad16) -> VCC
- U13 pad 8: unconnected-(U13-GND-Pad8) -> GND
- U14 pad 1: Net-(U14-S2) -> Net-(D18-A)
- U14 pad 15: Net-(U14-B2) -> Net-(U14-B3)
- U14 pad 16: unconnected-(U14-VCC-Pad16) -> VCC
- U14 pad 4: Net-(D18-A) -> Net-(D19-A)
- U14 pad 8: unconnected-(U14-GND-Pad8) -> GND
- U16 pad 3: Net-(U14-B2) -> Net-(U14-B3)
- U17 pad 10: unconnected-(U17-GND-Pad10) -> GND
- U17 pad 15: BUS_5 -> BUS_4
- U17 pad 17: BUS_5 -> BUS_6
- U17 pad 18: BUS_5 -> BUS_7
- U17 pad 20: unconnected-(U17-VCC-Pad20) -> VCC
- U17 pad 8: Net-(U14-S2) -> Net-(D18-A)
- U17 pad 9: Net-(D18-A) -> Net-(D19-A)
- U18 pad 1: BUS_5 -> /MAR/PROG
- U18 pad 10: BUS_5 -> /MAR/PROG
- U18 pad 11: BUS_5 -> /MAR/PROG
- U18 pad 13: BUS_5 -> /MAR/PROG
- U18 pad 14: BUS_5 -> /MAR/PROG
- U18 pad 16: unconnected-(U18-VCC-Pad16) -> VCC
- U18 pad 2: BUS_5 -> /MAR/PROG
- U18 pad 3: BUS_5 -> /MAR/PROG
- U18 pad 5: BUS_5 -> /MAR/PROG
- U18 pad 6: BUS_5 -> /MAR/PROG
- U18 pad 8: unconnected-(U18-GND-Pad8) -> GND
- U19 pad 16: unconnected-(U19-VCC-Pad16) -> VCC
- U19 pad 3: BUS_5 -> /MAR/PROG
- U19 pad 4: BUS_5 -> /MAR/PROG
- U19 pad 5: BUS_5 -> /MAR/PROG
- U19 pad 6: BUS_5 -> /MAR/PROG
- U19 pad 8: unconnected-(U19-GND-Pad8) -> GND
- U20 pad 12: Net-(U21-D2) -> Net-(U23-D0)
- U20 pad 13: Net-(U24-Zb) -> Net-(U24-Zd)
- U20 pad 2: Net-(U21-~{WE}) -> Net-(U21-*WE)
- U20 pad 3: Net-(U24-Zd) -> Net-(U24-Zb)
- U20 pad 4: Net-(U21-D0) -> Net-(U23-D3)
- U20 pad 5: Net-(U24-Zc) -> Net-(U24-Za)
- U20 pad 6: Net-(U21-D1) -> Net-(U23-D2)
- U20 pad 7: BUS_5 -> GND
- U20 pad 8: Net-(U23-D0) -> Net-(U21-D3)
- U20 pad 9: unconnected-(U20-Pad9) -> Net-(U52-Zd)
- U21 pad 11: Net-(U21-~{O}3) -> Net-(U21-*O3)
- U21 pad 2: BUS_5 -> GND
- U21 pad 3: Net-(U21-~{WE}) -> Net-(U21-*WE)
- U21 pad 5: Net-(U21-~{O}0) -> Net-(U21-*O0)
- U21 pad 7: Net-(U21-~{O}1) -> Net-(U21-*O1)
- U21 pad 8: BUS_5 -> GND
- U21 pad 9: Net-(U21-~{O}2) -> Net-(U21-*O2)
- U22 pad 10: (no net) -> unconnected-(U22-Pad10)
- U22 pad 11: (no net) -> unconnected-(U22-Pad11)
- U22 pad 12: (no net) -> unconnected-(U22-Pad12)
- U22 pad 13: (no net) -> unconnected-(U22-Pad13)
- U22 pad 2: Net-(U21-~{O}0) -> Net-(U21-D0)
- U22 pad 3: (no net) -> unconnected-(U22-Pad3)
- U22 pad 4: (no net) -> unconnected-(U22-Pad4)
- U22 pad 5: (no net) -> unconnected-(U22-Pad5)
- U22 pad 6: (no net) -> unconnected-(U22-Pad6)
- U22 pad 7: BUS_5 -> GND
- U22 pad 8: (no net) -> unconnected-(U22-Pad8)
- U22 pad 9: (no net) -> unconnected-(U22-Pad9)
- U23 pad 11: Net-(U23-~{O}3) -> Net-(U23-*O3)
- U23 pad 12: Net-(U21-~{O}0) -> Net-(U23-D3)
- U23 pad 2: BUS_5 -> GND
- U23 pad 3: Net-(U21-~{WE}) -> Net-(U21-*WE)
- U23 pad 5: Net-(U23-~{O}0) -> Net-(U23-*O0)
- U23 pad 6: Net-(U21-D0) -> Net-(U23-D1)
- U23 pad 7: Net-(U23-~{O}1) -> Net-(U23-*O1)
- U23 pad 8: BUS_5 -> GND
- U23 pad 9: Net-(U23-~{O}2) -> Net-(U23-*O2)
- U24 pad 1: BUS_5 -> /MAR/PROG
- U24 pad 15: BUS_5 -> GND
- U24 pad 8: BUS_5 -> GND
- U25 pad 10: BUS_5 -> GND
- U25 pad 15: BUS_5 -> BUS_4
- U25 pad 17: BUS_5 -> BUS_6
- U25 pad 18: BUS_5 -> BUS_7
- U26 pad 7: BUS_5 -> GND
- U27 pad 1: Net-(U23-~{O}0) -> Net-(U21-*O0)
- U27 pad 11: Net-(U21-~{WE}) -> Net-(U23-*O3)
- U27 pad 13: Net-(U21-~{O}1) -> Net-(U23-*O2)
- U27 pad 3: Net-(U23-~{O}1) -> Net-(U21-*O1)
- U27 pad 5: Net-(U23-~{O}2) -> Net-(U21-*O2)
- U27 pad 9: Net-(U23-~{O}3) -> Net-(U21-*O3)
- U28 pad 1: Net-(U21-~{O}2) -> Net-(U23-*O1)
- U28 pad 3: Net-(U21-~{O}3) -> Net-(U23-*O0)
- U28 pad 7: BUS_5 -> GND
- U29 pad 1: unconnected-(U29-A->B-Pad1) -> GND
- U33 pad 1: unconnected-(U33A-E-Pad1) -> GND
- U38 pad 13: BUS_5 -> BUS_4
- U38 pad 17: BUS_5 -> BUS_6
- U38 pad 18: BUS_5 -> BUS_7
- U4 pad 11: (no net) -> unconnected-(U4-Pad11)
- U4 pad 12: (no net) -> unconnected-(U4-Pad12)
- U4 pad 13: (no net) -> unconnected-(U4-Pad13)
- U41 pad 16: unconnected-(U41-VCC-Pad16) -> VCC
- U41 pad 8: unconnected-(U41-GND-Pad8) -> GND
- U42 pad 16: unconnected-(U42-VCC-Pad16) -> VCC
- U42 pad 8: unconnected-(U42-GND-Pad8) -> GND
- U47 pad 10: (no net) -> unconnected-(U47-Pad10)
- U47 pad 11: (no net) -> unconnected-(U47-Pad11)
- U47 pad 12: (no net) -> unconnected-(U47-Pad12)
- U47 pad 13: (no net) -> unconnected-(U47-Pad13)
- U47 pad 14: (no net) -> VCC
- U47 pad 5: (no net) -> unconnected-(U47-Pad5)
- U47 pad 6: (no net) -> unconnected-(U47-Pad6)
- U47 pad 7: (no net) -> GND
- U47 pad 8: (no net) -> unconnected-(U47-Pad8)
- U47 pad 9: (no net) -> unconnected-(U47-Pad9)
- U48 pad 10: unconnected-(U48-GND-Pad10) -> GND
- U48 pad 15: BUS_5 -> BUS_4
- U48 pad 17: BUS_5 -> BUS_6
- U48 pad 18: BUS_5 -> BUS_7
- U48 pad 2: /ALU/A_7 -> /ALU/A_4
- U48 pad 20: unconnected-(U48-VCC-Pad20) -> VCC
- U48 pad 3: /ALU/A_6 -> /ALU/A_5
- U48 pad 4: /ALU/A_5 -> /ALU/A_6
- U48 pad 5: /ALU/A_4 -> /ALU/A_7
- U48 pad 6: /ALU/A_3 -> /ALU/A_0
- U48 pad 7: /ALU/A_2 -> /ALU/A_1
- U48 pad 8: /ALU/A_1 -> /ALU/A_2
- U48 pad 9: /ALU/A_0 -> /ALU/A_3
- U49 pad 11: BUS_5 -> BUS_4
- U49 pad 13: BUS_5 -> BUS_6
- U49 pad 14: BUS_5 -> BUS_7
- U49 pad 16: unconnected-(U49-VCC-Pad16) -> VCC
- U49 pad 3: /ALU/A_4 -> /ALU/A_7
- U49 pad 4: /ALU/A_5 -> /ALU/A_6
- U49 pad 5: /ALU/A_6 -> /ALU/A_5
- U49 pad 6: /ALU/A_7 -> /ALU/A_4
- U49 pad 8: unconnected-(U49-GND-Pad8) -> GND
- U5 pad 10: Net-(U21-D3) -> Net-(U23-D1)
- U5 pad 11: Net-(U24-Za) -> Net-(U24-Zc)
- U5 pad 4: Net-(U23-D2) -> Net-(U21-D1)
- U5 pad 6: Net-(U21-D0) -> Net-(U21-D2)
- U50 pad 16: unconnected-(U50-VCC-Pad16) -> VCC
- U50 pad 3: /ALU/A_0 -> /ALU/A_3
- U50 pad 4: /ALU/A_1 -> /ALU/A_2
- U50 pad 5: /ALU/A_2 -> /ALU/A_1
- U50 pad 6: /ALU/A_3 -> /ALU/A_0
- U50 pad 8: unconnected-(U50-GND-Pad8) -> GND
- U51 pad 1: BUS_5 -> /MAR/PROG
- U51 pad 15: BUS_5 -> GND
- U51 pad 8: BUS_5 -> GND
- U52 pad 1: BUS_5 -> /MAR/PROG
- U52 pad 10: BUS_5 -> BUS_4
- U52 pad 11: BUS_5 -> Net-(U52-I0d)
- U52 pad 14: BUS_5 -> Net-(U52-I0c)
- U52 pad 15: BUS_5 -> GND
- U52 pad 2: BUS_5 -> Net-(U52-I0a)
- U52 pad 3: BUS_5 -> BUS_7
- U52 pad 5: BUS_5 -> Net-(U52-I0b)
- U52 pad 6: BUS_5 -> BUS_6
- U52 pad 8: BUS_5 -> GND
- U52 pad 9: Net-(U23-D0) -> Net-(U52-Zd)
- U6 pad 10: (no net) -> unconnected-(U6-Pad10)
- U6 pad 11: (no net) -> unconnected-(U6-Pad11)
- U6 pad 12: (no net) -> unconnected-(U6-Pad12)
- U6 pad 13: (no net) -> unconnected-(U6-Pad13)
- U6 pad 4: (no net) -> unconnected-(U6-Pad4)
- U6 pad 5: (no net) -> unconnected-(U6-Pad5)
- U6 pad 6: (no net) -> unconnected-(U6-Pad6)
- U6 pad 8: (no net) -> unconnected-(U6-Pad8)
- U6 pad 9: (no net) -> unconnected-(U6-Pad9)
- U7 pad 15: BUS_5 -> BUS_4
- U7 pad 17: BUS_5 -> BUS_6
- U7 pad 18: BUS_5 -> BUS_7
- U7 pad 2: /ALU/B_7 -> /ALU/B_4
- U7 pad 3: /ALU/B_6 -> /ALU/B_5
- U7 pad 4: /ALU/B_5 -> /ALU/B_6
- U7 pad 5: /ALU/B_4 -> /ALU/B_7
- U7 pad 6: /ALU/B_3 -> /ALU/B_0
- U7 pad 7: /ALU/B_2 -> /ALU/B_1
- U7 pad 8: /ALU/B_1 -> /ALU/B_2
- U7 pad 9: /ALU/B_0 -> /ALU/B_3
- U8 pad 11: BUS_5 -> BUS_4
- U8 pad 13: BUS_5 -> BUS_6
- U8 pad 14: BUS_5 -> BUS_7
- U8 pad 3: /ALU/B_4 -> /ALU/B_7
- U8 pad 4: /ALU/B_5 -> /ALU/B_6
- U8 pad 5: /ALU/B_6 -> /ALU/B_5
- U8 pad 6: /ALU/B_7 -> /ALU/B_4
- U9 pad 3: /ALU/B_0 -> /ALU/B_3
- U9 pad 4: /ALU/B_1 -> /ALU/B_2
- U9 pad 5: /ALU/B_2 -> /ALU/B_1
- U9 pad 6: /ALU/B_3 -> /ALU/B_0
Routing:
- net GND: track 0.00 -> 1804.2 mm, vias 0 -> 3
- net BUS_5: track 48.2 -> 0.00 mm
- net Net-(D30-K): track 0.00 -> 5.09 mm
- net Net-(D31-K): track 0.00 -> 4.90 mm
- net Net-(D26-K): track 0.00 -> 4.90 mm
- net Net-(D27-K): track 0.00 -> 4.88 mm
- net Net-(D33-K): track 0.00 -> 4.88 mm
- net Net-(D32-K): track 0.00 -> 4.69 mm
- net Net-(D29-K): track 0.00 -> 4.69 mm
- net Net-(D28-K): track 0.00 -> 4.69 mm
Other:
- copper layers 2 -> 6

Commit message: routed the traces for the ground plane.
Routing:
- net GND: track 1804.2 -> 1834.7 mm, vias 3 -> 5
Changed lines of the file:
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@@
+	)
+	(segment
+		(start 23.399 108.601)
+		(end 24.08 107.92)
+		(width 0.2)
+		(layer "F.Cu")
+		(net 1)
+	)
+	(segment
+		(start 24.08 107.92)
+		(end 24.5 107.92)
+		(width 0.2)
+		(layer "F.Cu")
+		(net 1)
+	)
+	(segment
+		(start 292.5 118.5)
+		(end 292.5073 118.5073)
+		(width 0.2)
+		(layer "F.Cu")
+		(net 1)
 	)
 	(segment
@@
 	)
 	(segment
+		(start 26 114)
+		(end 25.08 114)
+		(width 0.2)
+		(layer "F.Cu")
+		(net 1)
+	)
+	(segment
 		(start 196.4508 122.04)
 		(end 197.5 120.9908)
@@
 	)
 	(segment
+		(start 23.399 113.119)
+		(end 23.399 108.601)
+		(width 0.2)
+		(layer "F.Cu")
+		(net 1)
+	)
+	(segment
 		(start 290.5673 146.5673)
 		(end 292.5421 146.5673)
@@
 	)
 	(segment
+		(start 24.32 114.99)
+		(end 24.32 113.6)
+		(width 0.2)
+		(layer "F.Cu")
+		(net 1)
+	)
+	(segment
+		(start 24.5 113.42)
+		(end 23.7 113.42)
+		(width 0.2)
+		(layer "F.Cu")
+		(net 1)
+	)
+	(segment
 		(start 120.6998 151)
 		(end 120.8089 151.1091)
@@
 	)
 	(segment
+		(start 23.7 113.42)
+		(end 23.399 113.119)
+		(width 0.2)
+		(layer "F.Cu")
+		(net 1)
+	)
+	(segment
 		(start 284.4721 142.1873)
 		(end 286.3121 144.0273)
@@
 	)
 	(segment
+		(start 292.5073 118.5073)
+		(end 294.5921 118.5073)
+		(width 0.2)
+		(layer "F.Cu")
+		(net 1)
+	)
+	(segment
 		(start 189 115.5185)
 		(end 187.9015 114.42)
@@
 	)
 	(segment
+		(start 25.08 114)
+		(end 24.5 113.42)
+		(width 0.2)
+		(layer "F.Cu")
+		(net 1)
+	)
+	(segment
 		(start 285 140.5)
 		(end 285 141.6594)
@@
 		(start 196.42 114.42)
 		(end 196.04935 114.42)
+		(width 0.2)
+		(layer "F.Cu")
+		(net 1)
+	)
+	(segment
+		(start 24.32 113.6)
+		(end 24.5 113.42)
 		(width 0.2)
 		(layer "F.Cu")
@@
 	)
 	(via
+		(at 26 114)
+		(size 0.6)
+		(drill 0.3)
+		(layers "F.Cu" "B.Cu")
+		(net 1)
+	)
+	(via
+		(at 292.5 118.5)
+		(size 0.6)
+		(drill 0.3)
+		(layers "F.Cu" "B.Cu")
+		(net 1)
+	)
+	(via
 		(at 119 151)
 		(size 0.6)
@@
 	)
 	(segment
+		(start 27 114.99)
+		(end 26.99 114.99)
+		(width 0.2)
+		(layer "In1.Cu")
+		(net 1)
+	)
+	(segment
 		(start 89.44255 34.56)
 		(end 85.1198 34.56)
@@
 	)
 	(segment
+		(start 26.99 114.99)
+		(end 26 114)
+		(width 0.2)
+		(layer "In1.Cu")
+		(net 1)
+	)
+	(segment
 		(start 125.5 53.87995)
 		(end 124.00005 52.38)
@@
 	)
 	(segment
+		(start 38 112.42)
+		(end 35.43 114.99)
+		(width 0.2)
+		(layer "In1.Cu")
+		(net 1)
+	)
+	(segment
 		(start 277.4242 85.42)
 		(end 276.4755 86.3687)
@@
 	)
 	(segment
+		(start 281.9171 117.2223)
+		(end 291.5 117.2223)
+		(width 0.2)
+		(layer "In1.Cu")
+		(net 1)
+	)
+	(segment
 		(start 149.6664 117.3791)
 		(end 155.6664 117.3791)
@@
 	)
 	(segment
+		(start 291.5 117.5)
+		(end 292.5 118.5)
+		(width 0.2)
+		(layer "In1.Cu")
+		(net 1)
+	)
+	(segment
 		(start 189 138.8544)
 		(end 189 131.2344)
@@
 	)
 	(segment
+		(start 35.43 114.99)
+		(end 27 114.99)
+		(width 0.2)
+		(layer "In1.Cu")
+		(net 1)
+	)
+	(segment
 		(start 105.00005 44.72)
 		(end 106.5 43.22005)
@@
 	)
 	(segment
-		(start 281.9171 117.2223)
+		(start 291.5 117.2223)
 		(end 302.1271 117.2223)
 		(width 0.2)
@@
 	)
 	(segment
+		(start 291.5 117.2223)
+		(end 291.5 117.5)
+		(width 0.2)
+		(layer "In1.Cu")
+		(net 1)
+	)
+	(segment
 		(start 316.205 95.205)
 		(end 314.8 93.8)
@@
 		(width 0.2)
 		(layer "In1.Cu")
+		(net 1)
+	)
+	(segment
+		(start 27 114.99)
+		(end 24.32 114.99)
+		(width 0.2)
+		(layer "In1.Cu")

Commit message: finnished routing the PCB.
Routing:
- net VCC: track 0.00 -> 1340.6 mm, vias 0 -> 11
- net BUS_3: track 0.00 -> 557.5 mm, vias 0 -> 5
- net BUS_2: track 0.00 -> 550.3 mm, vias 0 -> 4
- net BUS_0: track 0.00 -> 542.2 mm, vias 0 -> 4
- net BUS_1: track 0.00 -> 530.0 mm, vias 0 -> 6
- net BUS_4: track 0.00 -> 485.6 mm, vias 0 -> 4
- net BUS_6: track 0.00 -> 484.8 mm, vias 0 -> 3
- net BUS_5: track 0.00 -> 484.1 mm, vias 0 -> 7
- net BUS_7: track 0.00 -> 460.3 mm, vias 0 -> 3
- net CLK: track 0.00 -> 380.8 mm, vias 0 -> 2
- net CLR: track 0.00 -> 360.7 mm, vias 0 -> 1
- net SU: track 0.00 -> 359.2 mm, vias 0 -> 1
- net HLT: track 0.00 -> 357.1 mm, vias 0 -> 2
- net GND: track 1834.7 -> 2135.1 mm
- net /MAR/PROG: track 0.00 -> 267.9 mm
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Other:
- board size 320.5 x 165.5 mm -> 320.5 x 157.5 mm
